Commit message: corrections1

File: src/gopigo3_description/urdf/gopigo3_v1.urdf (robot description, URDF)
Before this commit: robot gopigo, 3 links, 2 joints
Links:
- added link base_footprint
Joints:
- added joint base_link_joint: type fixed, parent base_footprint, child base_link, origin xyz=0 0 0.05 rpy=0 0 0

File: src/gopigo3_description/urdf/gopigo3_v2.urdf (robot description, URDF)
Before this commit: robot gopigo3, 8 links, 7 joints
Links:
- removed link base_scan
- removed link base_scan_solid
- added link base_footprint
- link base_link: geometry collision box size=0.5 0.5 0.25; collision sphere radius=0.075
- link camera: geometry collision box size=0.15 0.15 0.05; visual mesh filename=package://gopigo3_description/meshes/piCamera.stl scale=0.005 0.005 0.005
- link distance_sensor: geometry visual box size=0.01 0.01 0.01
- link distance_sensor_solid: geometry collision box size=0.01 0.01 0.01; visual mesh filename=package://gopigo3_description/meshes/IR_Sensor_Sharp_GP2Y_s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 scale=0.005 0.005 0.005
- link left_wheel: mass 0.15 -> 0.5; geometry collision cylinder length=0.1 radius=0.2; visual cylinder length=0.1 radius=0.2
- link right_wheel: mass 0.15 -> 0.5; geometry collision cylinder length=0.1 radius=0.2; visual cylinder length=0.1 radius=0.2
Joints:
- removed joint scan_joint
- removed joint scan_solid_joint
- added joint base_link_joint: type fixed, parent base_footprint, child base_link, origin xyz=0 0 0.05 rpy=0 0 0
- joint distance_sensor_joint: origin xyz=0.225 0 0.065 rpy=0 0 0 -> xyz=0.245 0 0.13 rpy=0 0 0
- joint joint_camera: origin xyz=0.25 0 0.025 rpy=0 0 0 -> xyz=0 0 0 rpy=0 0 0
- joint joint_left_wheel: origin xyz=0.1 0.15 0.0125 rpy=0 0 0 -> xyz=0.2 0.30 0.025 rpy=0 0 0
- joint joint_right_wheel: origin xyz=0.1 -0.15 0.0125 rpy=0 0 0 -> xyz=0.2 -0.30 0.025 rpy=0 0 0

File: src/gopigo3_description/urdf/gopigo3_v3.urdf (robot description, URDF)
Before this commit: robot gopigo3, 6 links, 5 joints
Links:
- added link base_footprint
- added link base_scan; visual box size=0.005 0.005 0.005
- added link base_scan_solid, mass 0.057; collision cylinder length=0.01575 radius=0.0275; visual mesh filename=package://gopigo3_description/meshes/X4.stl scale=0.002 0.002 0.002
- link base_link: geometry collision box size=0.5 0.25 0.125; collision sphere radius=0.025
- link camera: geometry collision box size=0.075 0.075 0.025; visual mesh filename=package://gopigo3_description/meshes/piCamera.stl scale=0.0025 0.0025 0.0025
- link distance_sensor: geometry visual box size=0.005 0.005 0.005
- link distance_sensor_solid: geometry collision box size=0.005 0.005 0.005; visual mesh filename=package://gopigo3_description/meshes/IR_Sensor_Sharp_GP2Y_s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 scale=0.0025 0.0025 0.0025
- link left_wheel: mass 0.5 -> 0.15; geometry collision cylinder length=0.05 radius=0.1; visual cylinder length=0.05 radius=0.1
- link right_wheel: mass 0.5 -> 0.15; geometry collision cylinder length=0.05 radius=0.1; visual cylinder length=0.05 radius=0.1
Joints:
- added joint base_link_joint: type fixed, parent base_footprint, child base_link, origin xyz=0 0 0.05 rpy=0 0 0
- added joint scan_joint: type fixed, parent base_link, child base_scan, origin xyz=0 0 0.125 rpy=0 0 3.14
- added joint scan_solid_joint: type fixed, parent base_scan, child base_scan_solid, origin xyz=0 0 0 rpy=0 0 0
- joint distance_sensor_joint: origin xyz=0.245 0 0.13 rpy=0 0 0 -> xyz=0.225 0 0.065 rpy=0 0 0
- joint joint_camera: origin xyz=0 0 0 rpy=0 0 0 -> xyz=0.25 0 0.025 rpy=0 0 0
- joint joint_left_wheel: origin xyz=0.2 0.30 0.025 rpy=0 0 0 -> xyz=0.1 0.15 0.0125 rpy=0 0 0
- joint joint_right_wheel: origin xyz=0.2 -0.30 0.025 rpy=0 0 0 -> xyz=0.1 -0.15 0.0125 rpy=0 0 0

File: src/gopigo3_description/urdf/gopigo3_v4.urdf (robot description, URDF)
Before this commit: robot gopigo3, 5 links, 4 joints
Links:
- added link base_footprint
Joints:
- added joint base_link_joint: type fixed, parent base_footprint, child base_link, origin xyz=0 0 0.05 rpy=0 0 0
