Commit message: SLAM with new model

File: src/gopigo3_description/urdf/gopigo3.urdf.xacro (robot description, xacro)
@@ -216,5 +216,5 @@
       <parent link="base_link"/>
       <child link="base_scan"/>
-      <origin xyz="-0.02 0 0.085" rpy="0 0 -1.57"/>
+      <origin xyz="-0.02 0 0.085" rpy="0 0 0"/>
       <!--LDS** origin xyz="-0.02 0 0.07" rpy="0 0 -1.6"/-->
     </joint>

Commit message: added tests

File: src/gopigo3_description/urdf/gopigo3.urdf.xacro (robot description, xacro)
@@ -4,6 +4,6 @@
   <xacro:include filename="$(find gopigo3_description)/urdf/gopigo3.gazebo.xacro"/>
   <xacro:property name="CADscale" value="0.0012" />
-  <!-- Which sensors to include -->
-<xacro:arg name="imu" default="false" />
+<!-- Which sensors to include -->
+<xacro:arg name="imu" default="true" />
 <!--xacro:property name="imu" value="true"/-->
 <xacro:arg name="distance"        default="true"/>

File: src/gopigo3_description/urdf/gopigo3_default.urdf (robot description, URDF)
Before this commit: robot gopigo3, 12 links, 11 joints
Links:
- removed link imu_link
Joints:
- removed joint imu_joint
