Commit message: Added laserscan

File: src/gopigo3_description/urdf/gopigo3.gazebo.xacro (robot description, xacro)
@@ -150,6 +150,8 @@
             <!--samples>360</samples>
             <resolution>1</resolution-->
-            <samples>500</samples>
-            <resolution>0.72</resolution>
+            <!--samples>500</samples-->
+            <!--resolution>0.72</resolution-->
+            <samples>720</samples>
+            <resolution>0.5</resolution>
             <min_angle>0.0</min_angle>
             <max_angle>6.28319</max_angle>

File: src/gopigo3_description/urdf/gopigo3.urdf.xacro (robot description, xacro)
@@ -6,5 +6,5 @@
 <!-- Which sensors to include -->
 <xacro:arg name="imu" default="true" />
-<!--xacro:property name="imu" value="true"/-->
+<xacro:property name="imu" value="true"/>
 <xacro:arg name="distance"        default="true"/>
 <xacro:arg name="pi_camera"       default="true"/>
