Commit message: Control corrections

File: src/gopigo3_description/urdf/gopigo3_stl.urdf (robot description, URDF)
Before this commit: robot gopigo3, 5 links, 4 joints
Links:
- added link base_footprint
- link base_scan: mass 0.057 -> 0.178; geometry collision cylinder length=0.05 radius=0.03; visual mesh filename=package://gopigo3_description/meshes/X4.stl scale=0.001158 0.001158 0.001158
Joints:
- added joint base_joint: type fixed, parent base_footprint, child base_link, origin xyz=0 0 0.016 rpy=0 0 0
- joint scan_joint: origin xyz=-0.01 0 0.11 rpy=0 0 0 -> xyz=0.02 0 0.11 rpy=0 0 0

Commit message: added bringup

File: src/gopigo3_description/urdf/gopigo3_stl.urdf (robot description, URDF)
Before this commit: robot gopigo3, 6 links, 5 joints
Links:
- link base_link: geometry collision box size=0.245 0.088 0.07; visual mesh filename=package://gopigo3_description/meshes/GoPiGo3_Body.stl scale=0.001158 0.001158 0.001158
- link left_wheel: mass 0.15 -> 0.032; geometry collision cylinder length=0.026 radius=0.033; visual mesh filename=package://gopigo3_description/meshes/GoPiGo3_Wheel.stl scale=0.001158 0.001158 0.001158
- link right_wheel: mass 0.15 -> 0.032; geometry collision cylinder length=0.026 radius=0.033; visual mesh filename=package://gopigo3_description/meshes/GoPiGo3_Wheel.stl scale=0.001158 0.001158 0.001158
Joints:
- joint base_joint: origin xyz=0 0 0.016 rpy=0 0 0 -> xyz=0 0 0.0 rpy=0 0 0
- joint joint_left_wheel: origin xyz=0.012 0.058 0.005 rpy=0 0 1.57 -> xyz=0 0.058 0.033 rpy=0 0 1.57
- joint joint_right_wheel: axis 1 0 0 -> -1 0 0; origin xyz=0.012 -0.058 0.005 rpy=0 0 -1.57 -> xyz=0 -0.058 0.033 rpy=0 0 -1.57
