Commit message: added hw gopigo3 corrections

File: src/gopigo3_description/urdf/gopigo3rp.urdf (robot description, URDF)
Before this commit: robot gopigo3, 12 links, 11 joints
Joints:
- joint scan_joint: origin xyz=-0.02 0 0.085 rpy=0 0 3.14 -> xyz=-0.02 0 0.085 rpy=0 0 0

Commit message: Bringup

File: src/gopigo3_description/urdf/gopigo3rp.urdf (robot description, URDF)
Before this commit: robot gopigo3, 12 links, 11 joints
Joints:
- joint scan_joint: origin xyz=-0.02 0 0.085 rpy=0 0 3.14 -> xyz=-0.02 0 0.085 rpy=0 0 3014

Commit message: Bringup

File: src/gopigo3_description/urdf/gopigo3rp.urdf (robot description, URDF)
Before this commit: robot gopigo3, 12 links, 11 joints
Joints:
- joint scan_joint: origin xyz=-0.02 0 0.085 rpy=0 0 3014 -> xyz=-0.02 0 0.085 rpy=0 0 3.14
