Commit message: model mpuig

File: src/gopigo3_description/urdf/gopigo3ydmpuig.urdf (robot description, URDF)
Before this commit: robot gopigo3, 8 links, 7 joints
Links:
- link base_link: geometry collision box size=0.2 0.1 0.05; visual mesh filename=package://gopigo3_description/meshes/GoPiGo3_Body2.stl scale=0.0012 0.0012 0.0012
- link camera_link: mass None -> 0.02
- link name_link: mass None -> 0.2
Joints:
- joint base_joint: origin xyz=0 0 0.075 rpy=0 0 0 -> xyz=0 0 0 rpy=0 0 0
- joint camera_joint: origin xyz=0.07 0 -0.02 rpy=0 0 0 -> xyz=0.07 0 0.03 rpy=0 0 0
- joint caster_back_joint: origin xyz=-0.132 0 -0.075 rpy=0 0 0 -> xyz=-0.132 0 0 rpy=0 0 0
- joint name_joint: origin xyz=-0.11 0 0.025 rpy=0 0 0 -> xyz=-0.115 0 0.057 rpy=0 0 0
- joint scan_joint: origin xyz=-0.008 0 0.085 rpy=0 0 0 -> xyz=0 0 0.14 rpy=0 0 0
- joint wheel_left_joint: origin xyz=0 0.058 -0.042 rpy=0 0 1.57 -> xyz=0 0.058 0.0 rpy=0 0 1.57
- joint wheel_right_joint: origin xyz=0 -0.058 -0.042 rpy=0 0 -1.57 -> xyz=0 -0.058 0.0 rpy=0 0 -1.57

Commit message: numbers added

File: src/gopigo3_description/urdf/gopigo3ydmpuig.urdf (robot description, URDF)
Before this commit: robot gopigo3, 8 links, 7 joints
Links:
- link base_link: geometry collision box size=0.245 0.088 0.02; visual mesh filename=package://gopigo3_description/meshes/GoPiGo3_Body2.stl scale=0.0012 0.0012 0.0012
- link name_link: geometry collision box size=0.01 0.01 0.002; visual mesh filename=package://gopigo3_description/meshes/number2.stl scale=0.0008 0.0008 0.0008
Joints:
- joint caster_back_joint: origin xyz=-0.132 0 0 rpy=0 0 0 -> xyz=-0.132 0 -0.04 rpy=0 0 0
