Commit message: corrections to model

File: src/gopigo3_description/urdf/gopigo3.urdf (robot description, URDF)
Before this commit: robot gopigo3, 12 links, 11 joints
Joints:
- joint camera_joint: origin xyz=0.04 0 0.04 rpy=0 0 0 -> xyz=0.07 0 -0.02 rpy=0 0 0

Commit message: model updated

File: src/gopigo3_description/urdf/gopigo3.urdf (robot description, URDF)
Before this commit: robot gopigo3, 12 links, 11 joints
Links:
- removed link base_link_cad
- removed link camera_rgb_frame
- removed link camera_rgb_optical_frame
- removed link distance_sensor
- removed link imu_link
- added link name_link, mass 0.2; collision box size=0.01 0.01 0.002; visual box size=0.01 0.03 0.02
- link base_link: geometry collision box size=0.245 0.088 0.02; visual mesh filename=package://gopigo3_description/meshes/GoPiGo3_Body2.stl scale=0.0012 0.0012 0.0012
- link camera_link: mass None -> 0.02
Joints:
- removed joint base_joint_cad
- removed joint camera_rgb_joint
- removed joint camera_rgb_optical_joint
- removed joint distance_sensor_joint
- removed joint imu_joint
- added joint name_joint: type fixed, parent base_link, child name_link, origin xyz=-0.14 0 0.07 rpy=0 0 0
- joint base_joint: origin xyz=0 0 0.075 rpy=0 0 0 -> xyz=0 0 0 rpy=0 0 0
- joint camera_joint: origin xyz=0.07 0 -0.02 rpy=0 0 0 -> xyz=0.07 0 0.03 rpy=0 0 0
- joint caster_back_joint: origin xyz=-0.132 0 -0.075 rpy=0 0 0 -> xyz=-0.132 0 -0.04 rpy=0 0 0
- joint scan_joint: origin xyz=-0.02 0 0.085 rpy=0 0 0 -> xyz=-0.02 0 0.14 rpy=0 0 0
- joint wheel_left_joint: origin xyz=0 0.058 -0.042 rpy=0 0 1.57 -> xyz=0 0.058 0.0 rpy=0 0 1.57
- joint wheel_right_joint: origin xyz=0 -0.058 -0.042 rpy=0 0 -1.57 -> xyz=0 -0.058 0.0 rpy=0 0 -1.57

File: src/gopigo3_description/urdf/gopigo3mpuig.urdf (robot description, URDF)
Before this commit: robot gopigo3, 8 links, 7 joints
Joints:
- joint scan_joint: origin xyz=0 0 0.14 rpy=0 0 0 -> xyz=-0.02 0 0.14 rpy=0 0 3.14
